File: input.kicad_sch (KiCad schematic)
At the start: 3 parts

Commit message: more work
Changed lines of the file:
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@@
 		(in_pos_files yes)
 		(dnp no)
-		(fields_autoplaced yes)
 		(property "Reference" "D4"
-			(at 58.42 41.6549 90)
+			(at 57.658 43.18 90)
 			(show_name no)
 			(do_not_autoplace no)
@@
 		(property "Value" "1N5819WS"
 			(at 58.42 44.1949 90)
+			(hide yes)
 			(show_name no)
 			(do_not_autoplace no)
@@
 		(in_pos_files yes)
 		(dnp no)
-		(fields_autoplaced yes)
 		(property "Reference" "D3"
-			(at 58.42 31.4949 90)
+			(at 57.404 33.02 90)
 			(show_name no)
 			(do_not_autoplace no)
@@
 		(property "Value" "1N5819WS"
 			(at 58.42 34.0349 90)
-			(show_name no)
-			(do_not_autoplace no)
+			(hide yes)
+			(show_name no)
+			(do_not_autoplace no)
