File: pandahat.kicad_sch (KiCad schematic)
At the start: 6 parts, among them J1 GPIO, J19 Conn_01x03

Commit message: more work
Connections:
- net UART_RX: now also J19.2 (Pin_2); no longer J19.3 (Pin_3)
- net UART_TX: now also J19.3 (Pin_3); no longer J19.2 (Pin_2)
Changed lines of the file:
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@@
+	)
+	(junction
+		(at 58.42 58.42)
+		(diameter 1.016)
+		(color 0 0 0 0)
+	)
+	(junction
+		(at 76.2 68.58)
+		(diameter 1.016)
+		(color 0 0 0 0)
+	)
+	(junction
+		(at 76.2 63.5)
+		(diameter 1.016)
+		(color 0 0 0 0)
+	)
+	(junction
+		(at 76.2 50.8)
+		(diameter 1.016)
+		(color 0 0 0 0)
 	)
 	(junction
@@
 		(color 0 0 0 0)
 	)
-	(junction
-		(at 58.42 58.42)
-		(diameter 1.016)
-		(color 0 0 0 0)
-	)
-	(junction
-		(at 76.2 68.58)
-		(diameter 1.016)
-		(color 0 0 0 0)
-	)
-	(junction
-		(at 76.2 63.5)
-		(diameter 1.016)
-		(color 0 0 0 0)
-	)
-	(junction
-		(at 76.2 50.8)
-		(diameter 1.016)
-		(color 0 0 0 0)
-	)
 	(wire
 		(pts
@@
 	(wire
 		(pts
-			(xy 101.6 35.56) (xy 101.6 19.05)
-		)
-		(stroke
-			(width 0)
-			(type default)
-		)
-	)
-	(wire
-		(pts
 			(xy 73.66 76.2) (xy 100.33 76.2)
 		)
@@
 	(wire
 		(pts
-			(xy 104.14 21.59) (xy 107.95 21.59)
-		)
-		(stroke
-			(width 0)
-			(type default)
-		)
-	)
-	(wire
-		(pts
 			(xy 60.96 30.48) (xy 31.75 30.48)
 		)
@@
 	(wire
 		(pts
+			(xy 101.6 35.56) (xy 101.6 21.59)
+		)
+		(stroke
+			(width 0)
+			(type default)
+		)
+	)
+	(wire
+		(pts
 			(xy 31.75 35.56) (xy 60.96 35.56)
 		)
@@
 	(wire
 		(pts
+			(xy 104.14 19.05) (xy 104.14 38.1)
+		)
+		(stroke
+			(width 0)
+			(type default)
+		)
+	)
+	(wire
+		(pts
+			(xy 73.66 38.1) (xy 104.14 38.1)
+		)
+		(stroke
+			(width 0)
+			(type default)
+		)
+	)
+	(wire
+		(pts
+			(xy 31.75 71.12) (xy 60.96 71.12)
+		)
+		(stroke
+			(width 0)
+			(type solid)
+		)
+	)
+	(wire
+		(pts
+			(xy 73.66 71.12) (xy 100.33 71.12)
+		)
+		(stroke
+			(width 0)
+			(type solid)
+		)
+	)
+	(wire
+		(pts
+			(xy 73.66 66.04) (xy 100.33 66.04)
+		)
+		(stroke
+			(width 0)
+			(type solid)
+		)
+	)
+	(wire
+		(pts
+			(xy 58.42 76.2) (xy 60.96 76.2)
+		)
+		(stroke
+			(width 0)
+			(type solid)
+		)
+	)
+	(wire
+		(pts
+			(xy 73.66 73.66) (xy 100.33 73.66)
+		)
+		(stroke
+			(width 0)
+			(type solid)
+		)
+	)
+	(wire
+		(pts
+			(xy 76.2 33.02) (xy 73.66 33.02)
+		)
+		(stroke
+			(width 0)
+			(type solid)
+		)
+	)
+	(wire
+		(pts
+			(xy 31.75 73.66) (xy 60.96 73.66)
+		)
+		(stroke
+			(width 0)
+			(type solid)
+		)
+	)
+	(wire
+		(pts
 			(xy 73.66 35.56) (xy 101.6 35.56)
 		)
@@
 	(wire
 		(pts
-			(xy 73.66 38.1) (xy 104.14 38.1)
-		)
-		(stroke
-			(width 0)
-			(type default)
-		)
-	)
-	(wire
-		(pts
-			(xy 31.75 71.12) (xy 60.96 71.12)
-		)
-		(stroke
-			(width 0)
-			(type solid)
-		)
-	)
-	(wire
-		(pts
-			(xy 73.66 71.12) (xy 100.33 71.12)
-		)
-		(stroke
-			(width 0)
-			(type solid)
-		)
-	)
-	(wire
-		(pts
-			(xy 73.66 66.04) (xy 100.33 66.04)
-		)
-		(stroke
-			(width 0)
-			(type solid)
-		)
-	)
-	(wire
-		(pts
-			(xy 58.42 76.2) (xy 60.96 76.2)
-		)
-		(stroke
-			(width 0)
-			(type solid)
-		)
-	)
-	(wire
-		(pts
-			(xy 73.66 73.66) (xy 100.33 73.66)
-		)
-		(stroke
-			(width 0)
-			(type solid)
-		)
-	)
-	(wire
-		(pts
-			(xy 76.2 33.02) (xy 73.66 33.02)
-		)
-		(stroke
-			(width 0)
-			(type solid)
-		)
-	)
-	(wire
-		(pts
-			(xy 31.75 73.66) (xy 60.96 73.66)
-		)
-		(stroke
-			(width 0)
-			(type solid)
-		)
-	)
-	(wire
-		(pts
 			(xy 101.6 35.56) (xy 113.03 35.56)
 		)
@@
 	(wire
 		(pts
-			(xy 101.6 19.05) (xy 107.95 19.05)
-		)
-		(stroke
-			(width 0)
-			(type default)
-		)
-	)
-	(wire
-		(pts
 			(xy 76.2 68.58) (xy 76.2 80.01)
 		)
@@
 	(wire
 		(pts
-			(xy 104.14 38.1) (xy 104.14 21.59)
+			(xy 104.14 19.05) (xy 107.95 19.05)
 		)
 		(stroke
@@
 		)
 	)
+	(wire
+		(pts
+			(xy 101.6 21.59) (xy 107.95 21.59)
+		)
+		(stroke
+			(width 0)
+			(type default)
+		)
+	)
