File: untitled.kicad_sch (KiCad schematic)
At the start: 34 parts, among them CN7 Wago connector, J12 Conn_01x03, Q1 MMBT3904-C20526, Q2 AO3401A, U1 AMS1117-3.3, U2 LM2596-5.0FW05ARHQ, U4 CJ431_C3113

Commit message: more work
Parts:
- removed L2: FXL0630-6R8-M, easyeda2kicad:IND-SMD_L7.0-W6.6, symbol lol:FXL0630-6R8-M
- added D29: SS54_C22452, easyeda2kicad:SMA_L4.4-W2.8-LS5.4-R-RD, symbol lol:SS54_C22452
- added L2: 47uH, easyeda2kicad:IND-SMD_L7.2-W6.6_GPSR07X0, symbol lol:CYA0650-47UH
Connections:
- net +5V: now also L2.2
- net +BATT: now also D1.2
- net VPP: now also D29.1 (A); no longer C2.1, C3.1, D1.2, U2.1 (VIN)
- net at D2.2 (K), U2.2 (Output): now also L2.1
- new net: C2.1, C3.1, D29.2 (K), U2.1 (VIN)
Other:
- moved on the sheet: D1
